Commit message: synchronize Rviz and Gazebo

File: irb6640_description/urdf/irb6640.xacro (robot description, xacro)
@@ -5,10 +5,4 @@
   <xacro:include filename="$(find irb6640_description)/urdf/irb6640.gazebo" />
   <xacro:include filename="$(find abb_resources)/urdf/common_materials.xacro"/>
-    <!-- Used for fixing robot to Gazebo ground -->
-    <link name="world"/>
-    <joint name="fixed" type="fixed">
-      <parent link="world"/>
-      <child link="base_link"/>
-    </joint>
     <!-- link list -->
     <link name="base_link">
@@ -303,10 +297,10 @@
    <!-- end of joint list -->
     <!-- ROS base_link to ABB World Coordinates transform -->
-<!--    <link name="base" />
+    <link name="base" />
     <joint name="base_link-base" type="fixed">
       <origin xyz="0 0 0" rpy="0 0 0"/>
       <parent link="base_link"/>
       <child link="base"/>
-    </joint> -->
+    </joint>
    <!-- transmission list -->
    <transmission name="tran1">
@@ -316,5 +310,4 @@
      </joint>
      <actuator name="motor1">
-       <hardwareInterface>hardware_interface/PositionJointInterface</hardwareInterface>
        <mechanicalReduction>1</mechanicalReduction>
      </actuator>
@@ -326,5 +319,4 @@
      </joint>
      <actuator name="motor2">
-       <hardwareInterface>hardware_interface/PositionJointInterface</hardwareInterface>
        <mechanicalReduction>1</mechanicalReduction>
      </actuator>
@@ -336,5 +328,4 @@
      </joint>
      <actuator name="motor3">
-       <hardwareInterface>hardware_interface/PositionJointInterface</hardwareInterface>
        <mechanicalReduction>1</mechanicalReduction>
      </actuator>
@@ -346,5 +337,4 @@
      </joint>
      <actuator name="motor4">
-       <hardwareInterface>hardware_interface/PositionJointInterface</hardwareInterface>
        <mechanicalReduction>1</mechanicalReduction>
      </actuator>
@@ -356,5 +346,4 @@
      </joint>
      <actuator name="motor5">
-       <hardwareInterface>hardware_interface/PositionJointInterface</hardwareInterface>
        <mechanicalReduction>1</mechanicalReduction>
      </actuator>
@@ -366,8 +355,13 @@
      </joint>
      <actuator name="motor6">
-       <hardwareInterface>hardware_interface/PositionJointInterface</hardwareInterface>
        <mechanicalReduction>1</mechanicalReduction>
      </actuator>
    </transmission>
   <!-- end of transmission list -->
+  <!-- Fix robot to Gazebo world -->
+  <link name="world"/>
+  <joint name="world-base_link-fixed" type="fixed">
+    <parent link="world"/>
+    <child link="base_link"/>
+  </joint>
 </robot>

Commit message: add overhead cameras

File: irb6640_description/urdf/irb6640.xacro (robot description, xacro)
@@ -155,4 +155,7 @@
     <link name="tool0"/>
     <link name="camera_link_optical"/>
+    <link name="world_camera_link_optical_1"/>
+    <link name="world_camera_link_optical_2"/>
+    <link name="world_camera_link_optical_3"/>
     <!--Cylinder and piston -->
     <link name="link_cylinder">
@@ -198,5 +201,5 @@
       </inertial>
     </link>
-    <!-- Camera -->
+    <!-- Camera on the wrist -->
     <link name="camera_link">
       <collision>
@@ -212,4 +215,65 @@
         </geometry>
         <material name="red"/>
+      </visual>
+      <inertial>
+        <mass value="1e-5" />
+        <origin xyz="0 0 0" rpy="0 0 0"/>
+        <inertia ixx="1e-6" ixy="0" ixz="0" iyy="1e-6" iyz="0" izz="1e-6" />
+      </inertial>
+    </link>
+    <!-- Cameras overhead -->
+    <link name="world_camera_1">
+      <collision>
+        <origin xyz="0 0 0" rpy="0 0 0"/>
+        <geometry>
+	  <box size="${camera_link} ${camera_link} ${camera_link}"/>
+        </geometry>
+      </collision>
+      <visual>
+        <origin xyz="0 0 0" rpy="0 0 0"/>
+        <geometry>
+	<box size="${camera_link} ${camera_link} ${camera_link}"/>
+        </geometry>
+        <material name="red"/>
+      </visual>
+      <inertial>
+        <mass value="1e-5" />
+        <origin xyz="0 0 0" rpy="0 0 0"/>
+        <inertia ixx="1e-6" ixy="0" ixz="0" iyy="1e-6" iyz="0" izz="1e-6" />
+      </inertial>
+    </link>
+    <link name="world_camera_2">
+      <collision>
+        <origin xyz="0 0 0" rpy="0 0 0"/>
+        <geometry>
+	  <box size="${camera_link} ${camera_link} ${camera_link}"/>
+        </geometry>
+      </collision>
+      <visual>
+        <origin xyz="0 0 0" rpy="0 0 0"/>
+        <geometry>
+	<box size="${camera_link} ${camera_link} ${camera_link}"/>
+        </geometry>
+        <material name="blue"/>
+      </visual>
+      <inertial>
+        <mass value="1e-5" />
+        <origin xyz="0 0 0" rpy="0 0 0"/>
+        <inertia ixx="1e-6" ixy="0" ixz="0" iyy="1e-6" iyz="0" izz="1e-6" />
+      </inertial>
+    </link>
+     <link name="world_camera_3">
+      <collision>
+        <origin xyz="0 0 0" rpy="0 0 0"/>
+        <geometry>
+	  <box size="${camera_link} ${camera_link} ${camera_link}"/>
+        </geometry>
+      </collision>
+      <visual>
+        <origin xyz="0 0 0" rpy="0 0 0"/>
+        <geometry>
+	<box size="${camera_link} ${camera_link} ${camera_link}"/>
+        </geometry>
+        <material name="blue"/>
       </visual>
       <inertial>
@@ -288,4 +352,22 @@
      <child link="camera_link"/>
    </joint>
+   <joint name="world_camera_joint_1" type="fixed">
+     <axis xyz="0 1 0" />
+     <origin xyz="1 0 3" rpy="0 1.57 0"/>
+     <parent link="base_link"/>
+     <child link="world_camera_1"/>
+   </joint>
+   <joint name="world_camera_joint_2" type="fixed">
+     <axis xyz="0 1 0" />
+     <origin xyz="0 1 0" rpy="0 0 0"/>
+     <parent link="world_camera_1"/>
+     <child link="world_camera_2"/>
+   </joint>
+   <joint name="world_camera_joint_3" type="fixed">
+     <axis xyz="0 1 0" />
+     <origin xyz="0 -1 0" rpy="0 0 0"/>
+     <parent link="world_camera_1"/>
+     <child link="world_camera_3"/>
+   </joint>
    <joint name="camera_optical_joint" type="fixed">
      <!-- these values have to be these values otherwise the gazebo camera image
@@ -294,4 +376,25 @@
      <parent link="camera_link"/>
      <child link="camera_link_optical"/>
+   </joint>
+   <joint name="world_camera_optical_joint_1" type="fixed">
+     <!-- these values have to be these values otherwise the gazebo camera image
+        won't be aligned properly with the frame it is supposedly originating from -->
+     <origin xyz="0 0 0" rpy="-1.57 0 -1.57"/>
+     <parent link="world_camera_1"/>
+     <child link="world_camera_link_optical_1"/>
+   </joint>
+   <joint name="world_camera_optical_joint_2" type="fixed">
+     <!-- these values have to be these values otherwise the gazebo camera image
+        won't be aligned properly with the frame it is supposedly originating from -->
+     <origin xyz="0 0 0" rpy="-1.57 0 -1.57"/>
+     <parent link="world_camera_2"/>
+     <child link="world_camera_link_optical_2"/>
+   </joint>
+   <joint name="world_camera_optical_joint_3" type="fixed">
+     <!-- these values have to be these values otherwise the gazebo camera image
+        won't be aligned properly with the frame it is supposedly originating from -->
+     <origin xyz="0 0 0" rpy="-1.57 0 -1.57"/>
+     <parent link="world_camera_3"/>
+     <child link="world_camera_link_optical_3"/>
    </joint>
    <!-- end of joint list -->

Commit message: update robot model to include vacuum gripper

File: irb6640_description/urdf/irb6640.xacro (robot description, xacro)
@@ -151,4 +151,24 @@
         <origin rpy="0 0 0" xyz="0.019851 -0.000031 0.001144"/>
         <inertia ixx="0.039" ixy="0" ixz="0" iyy="0.0234" iyz="0" izz="0.0234"/>
+      </inertial>
+    </link>
+    <link name="vacuum_gripper">
+      <gravity>0</gravity>
+      <collision name="collision">
+        <origin xyz="0 0 0" rpy="0 0 0"/>
+        <geometry>
+          <mesh filename="package://irb6640_gazebo/models/vacuum_gripper.dae" scale="0.3048 0.3048 0.3048"/>
+        </geometry>
+      </collision>
+      <visual name="visual">
+        <origin xyz="0 0 0" rpy="0 0 0"/>
+        <geometry>
+          <mesh filename="package://irb6640_gazebo/models/vacuum_gripper.dae" scale="0.3048 0.3048 0.3048"/>
+        </geometry>
+      </visual>
+      <inertial>
+        <mass value="1"/>
+        <origin rpy="0 0 0" xyz="0 0 0"/>
+        <inertia ixx="1" ixy="0" ixz="0" iyy="1" iyz="0" izz="1"/>
       </inertial>
     </link>
@@ -327,8 +347,14 @@
       <limit effort="100" lower="-6.283" upper="6.283" velocity="3.3161"/>
    </joint>
-   <joint name="joint_6-tool0" type="fixed">
+   <joint name="joint_6_tool0" type="fixed">
      <parent link="link_6"/>
      <child link="tool0"/>
      <origin rpy="0 1.57079632679 0" xyz="0 0 0"/>
+   </joint>
+   <joint name="link_6_vacuum_gripper" type="revolute">
+     <parent link="link_6"/>
+     <child link="vacuum_gripper"/>
+     <origin rpy="0 -1.57079632679 0" xyz="0.295 0 0"/>
+     <limit effort="30" velocity="1.0" lower="0" upper="0" />
    </joint>
    <joint name="joint_cylinder" type="continuous">
@@ -348,5 +374,5 @@
    <joint name="camera_joint" type="fixed">
      <axis xyz="0 1 0" />
-     <origin xyz="${camera_link} 0 0" rpy="0 0 0"/>
+     <origin xyz="0.15 0 0" rpy="0 0 0"/>
      <parent link="link_6"/>
      <child link="camera_link"/>
@@ -354,5 +380,5 @@
    <joint name="world_camera_joint_1" type="fixed">
      <axis xyz="0 1 0" />
-     <origin xyz="1 0 3" rpy="0 1.57 0"/>
+     <origin xyz="0 0 2.6" rpy="0 1.57 0"/>
      <parent link="base_link"/>
      <child link="world_camera_1"/>
@@ -360,5 +386,5 @@
    <joint name="world_camera_joint_2" type="fixed">
      <axis xyz="0 1 0" />
-     <origin xyz="0 1 0" rpy="0 0 0"/>
+     <origin xyz="0 1.5 0" rpy="0 0 0"/>
      <parent link="world_camera_1"/>
      <child link="world_camera_2"/>
@@ -366,5 +392,5 @@
    <joint name="world_camera_joint_3" type="fixed">
      <axis xyz="0 1 0" />
-     <origin xyz="0 -1 0" rpy="0 0 0"/>
+     <origin xyz="0 -1.5 0" rpy="0 0 0"/>
      <parent link="world_camera_1"/>
      <child link="world_camera_3"/>
@@ -461,8 +487,17 @@
      </actuator>
    </transmission>
+   <transmission name="tran7">
+     <type>transmission_interface/SimpleTransmission</type>
+     <joint name="link_6_vacuum_gripper">
+       <hardwareInterface>hardware_interface/PositionJointInterface</hardwareInterface>
+     </joint>
+     <actuator name="motor7">
+       <mechanicalReduction>1</mechanicalReduction>
+     </actuator>
+   </transmission>
   <!-- end of transmission list -->
   <!-- Fix robot to Gazebo world -->
   <link name="world"/>
-  <joint name="world-base_link-fixed" type="fixed">
+  <joint name="world_base_link-fixed" type="fixed">
     <parent link="world"/>
     <child link="base_link"/>

Commit message: make vacuum gripper working more robustly; lots of changes

File: irb6640_description/urdf/irb6640.xacro (robot description, xacro)
@@ -154,15 +154,14 @@
     </link>
     <link name="vacuum_gripper">
-      <gravity>0</gravity>
-      <collision name="collision">
-        <origin xyz="0 0 0" rpy="0 0 0"/>
-        <geometry>
-          <mesh filename="package://irb6640_gazebo/models/vacuum_gripper.dae" scale="0.3048 0.3048 0.3048"/>
-        </geometry>
-      </collision>
-      <visual name="visual">
-        <origin xyz="0 0 0" rpy="0 0 0"/>
-        <geometry>
-          <mesh filename="package://irb6640_gazebo/models/vacuum_gripper.dae" scale="0.3048 0.3048 0.3048"/>
+      <collision name="collision">
+        <origin xyz="0 0 0" rpy="0 0 0"/>
+        <geometry>
+          <mesh filename="package://irb6640_gazebo/models/vacuum_gripper.dae" scale="0.8 0.8 0.8"/>
+        </geometry>
+      </collision>
+      <visual name="visual">
+        <origin xyz="0 0 0" rpy="0 0 0"/>
+        <geometry>
+          <mesh filename="package://irb6640_gazebo/models/vacuum_gripper.dae" scale="0.8 0.8 0.8"/>
         </geometry>
       </visual>
@@ -170,5 +169,5 @@
         <mass value="1"/>
         <origin rpy="0 0 0" xyz="0 0 0"/>
-        <inertia ixx="1" ixy="0" ixz="0" iyy="1" iyz="0" izz="1"/>
+        <inertia ixx="0.1" ixy="0" ixz="0" iyy="0.1" iyz="0" izz="0.1"/>
       </inertial>
     </link>
@@ -226,5 +225,5 @@
         <origin xyz="0 0 0" rpy="0 0 0"/>
         <geometry>
-	  <box size="${camera_link} ${camera_link} ${camera_link}"/>
+	      <box size="${camera_link} ${camera_link} ${camera_link}"/>
         </geometry>
       </collision>
@@ -232,5 +231,5 @@
         <origin xyz="0 0 0" rpy="0 0 0"/>
         <geometry>
-	<box size="${camera_link} ${camera_link} ${camera_link}"/>
+	      <box size="${camera_link} ${camera_link} ${camera_link}"/>
         </geometry>
         <material name="red"/>
@@ -247,5 +246,5 @@
         <origin xyz="0 0 0" rpy="0 0 0"/>
         <geometry>
-	  <box size="${camera_link} ${camera_link} ${camera_link}"/>
+          <mesh filename="package://irb6640_gazebo/models/camera.dae" scale="0.5 0.5 0.5"/>
         </geometry>
       </collision>
@@ -253,7 +252,6 @@
         <origin xyz="0 0 0" rpy="0 0 0"/>
         <geometry>
-	<box size="${camera_link} ${camera_link} ${camera_link}"/>
-        </geometry>
-        <material name="red"/>
+	      <mesh filename="package://irb6640_gazebo/models/camera.dae" scale="0.5 0.5 0.5"/>
+        </geometry>
       </visual>
       <inertial>
@@ -267,5 +265,5 @@
         <origin xyz="0 0 0" rpy="0 0 0"/>
         <geometry>
-	  <box size="${camera_link} ${camera_link} ${camera_link}"/>
+	      <mesh filename="package://irb6640_gazebo/models/camera.dae" scale="0.5 0.5 0.5"/>
         </geometry>
       </collision>
@@ -273,7 +271,6 @@
         <origin xyz="0 0 0" rpy="0 0 0"/>
         <geometry>
-	<box size="${camera_link} ${camera_link} ${camera_link}"/>
-        </geometry>
-        <material name="blue"/>
+	      <mesh filename="package://irb6640_gazebo/models/camera.dae" scale="0.5 0.5 0.5"/>
+        </geometry>
       </visual>
       <inertial>
@@ -287,5 +284,5 @@
         <origin xyz="0 0 0" rpy="0 0 0"/>
         <geometry>
-	  <box size="${camera_link} ${camera_link} ${camera_link}"/>
+	      <mesh filename="package://irb6640_gazebo/models/camera.dae" scale="0.5 0.5 0.5"/>
         </geometry>
       </collision>
@@ -293,7 +290,6 @@
         <origin xyz="0 0 0" rpy="0 0 0"/>
         <geometry>
-	<box size="${camera_link} ${camera_link} ${camera_link}"/>
-        </geometry>
-        <material name="blue"/>
+	      <mesh filename="package://irb6640_gazebo/models/camera.dae" scale="0.5 0.5 0.5"/>
+        </geometry>
       </visual>
       <inertial>
@@ -346,83 +342,83 @@
       <child link="link_6"/>
       <limit effort="100" lower="-6.283" upper="6.283" velocity="3.3161"/>
-   </joint>
-   <joint name="joint_6_tool0" type="fixed">
-     <parent link="link_6"/>
-     <child link="tool0"/>
-     <origin rpy="0 1.57079632679 0" xyz="0 0 0"/>
-   </joint>
-   <joint name="link_6_vacuum_gripper" type="revolute">
-     <parent link="link_6"/>
-     <child link="vacuum_gripper"/>
-     <origin rpy="0 -1.57079632679 0" xyz="0.295 0 0"/>
-     <limit effort="30" velocity="1.0" lower="0" upper="0" />
-   </joint>
-   <joint name="joint_cylinder" type="continuous">
-     <origin rpy="0 0 0" xyz="-0.3647 0 -0.1455"/>
-     <axis xyz="0 1 0"/>
-     <parent link="link_1"/>
-     <child link="link_cylinder"/>
-     <mimic joint="joint_2" multiplier="-0.25"/>
-   </joint>
-   <joint name="joint_piston" type="continuous">
-     <origin rpy="0 0 0" xyz="-0.22 0 -0.0672"/>
-     <axis xyz="0 1 0"/>
-     <parent link="link_2"/>
-     <child link="link_piston"/>
-     <mimic joint="joint_2" multiplier="-1.25"/>
-   </joint>
-   <joint name="camera_joint" type="fixed">
-     <axis xyz="0 1 0" />
-     <origin xyz="0.15 0 0" rpy="0 0 0"/>
-     <parent link="link_6"/>
-     <child link="camera_link"/>
-   </joint>
-   <joint name="world_camera_joint_1" type="fixed">
-     <axis xyz="0 1 0" />
-     <origin xyz="0 0 2.6" rpy="0 1.57 0"/>
-     <parent link="base_link"/>
-     <child link="world_camera_1"/>
-   </joint>
-   <joint name="world_camera_joint_2" type="fixed">
-     <axis xyz="0 1 0" />
-     <origin xyz="0 1.5 0" rpy="0 0 0"/>
-     <parent link="world_camera_1"/>
-     <child link="world_camera_2"/>
-   </joint>
-   <joint name="world_camera_joint_3" type="fixed">
-     <axis xyz="0 1 0" />
-     <origin xyz="0 -1.5 0" rpy="0 0 0"/>
-     <parent link="world_camera_1"/>
-     <child link="world_camera_3"/>
-   </joint>
-   <joint name="camera_optical_joint" type="fixed">
-     <!-- these values have to be these values otherwise the gazebo camera image
+    </joint>
+    <joint name="joint_6_tool0" type="fixed">
+      <parent link="link_6"/>
+      <child link="tool0"/>
+      <origin rpy="0 1.57079632679 0" xyz="0 0 0"/>
+    </joint>
+    <joint name="link_6_vacuum_gripper" type="revolute">
+      <parent link="link_6"/>
+      <child link="vacuum_gripper"/>
+      <origin rpy="0 -1.57079632679 0" xyz="0.12 0 0"/>
+      <limit effort="30" velocity="1.0" lower="0" upper="0" />
+    </joint>
+    <joint name="joint_cylinder" type="continuous">
+      <origin rpy="0 0 0" xyz="-0.3647 0 -0.1455"/>
+      <axis xyz="0 1 0"/>
+      <parent link="link_1"/>
+      <child link="link_cylinder"/>
+      <mimic joint="joint_2" multiplier="-0.25"/>
+    </joint>
+    <joint name="joint_piston" type="continuous">
+      <origin rpy="0 0 0" xyz="-0.22 0 -0.0672"/>
+      <axis xyz="0 1 0"/>
+      <parent link="link_2"/>
+      <child link="link_piston"/>
+      <mimic joint="joint_2" multiplier="-1.25"/>
+    </joint>
+    <joint name="camera_joint" type="fixed">
+      <axis xyz="0 1 0" />
+      <origin xyz="-0.15 0 0" rpy="0 0 0"/>
+      <parent link="link_6"/>
+      <child link="camera_link"/>
+    </joint>
+    <joint name="world_camera_joint_1" type="fixed">
+      <axis xyz="0 1 0" />
+      <origin xyz="0 0 2.5" rpy="0 1.57 0"/>
+      <parent link="base_link"/>
+      <child link="world_camera_1"/>
+    </joint>
+    <joint name="world_camera_joint_2" type="fixed">
+      <axis xyz="0 1 0" />
+      <origin xyz="0 1.5 0" rpy="0 0 0"/>
+      <parent link="world_camera_1"/>
+      <child link="world_camera_2"/>
+    </joint>
+    <joint name="world_camera_joint_3" type="fixed">
+      <axis xyz="0 1 0" />
+      <origin xyz="0 -1.5 0" rpy="0 0 0"/>
+      <parent link="world_camera_1"/>
+      <child link="world_camera_3"/>
+    </joint>
+    <joint name="camera_optical_joint" type="fixed">
+      <!-- these values have to be these values otherwise the gazebo camera image
         won't be aligned properly with the frame it is supposedly originating from -->
-     <origin xyz="0 0 0" rpy="-1.57 0 -1.57"/>
-     <parent link="camera_link"/>
-     <child link="camera_link_optical"/>
-   </joint>
-   <joint name="world_camera_optical_joint_1" type="fixed">
-     <!-- these values have to be these values otherwise the gazebo camera image
+      <origin xyz="0 0 0" rpy="-1.57 0 -1.57"/>
+      <parent link="camera_link"/>
+      <child link="camera_link_optical"/>
+    </joint>
+    <joint name="world_camera_optical_joint_1" type="fixed">
+      <!-- these values have to be these values otherwise the gazebo camera image
         won't be aligned properly with the frame it is supposedly originating from -->
-     <origin xyz="0 0 0" rpy="-1.57 0 -1.57"/>
-     <parent link="world_camera_1"/>
-     <child link="world_camera_link_optical_1"/>
-   </joint>
-   <joint name="world_camera_optical_joint_2" type="fixed">
-     <!-- these values have to be these values otherwise the gazebo camera image
+      <origin xyz="0 0 0" rpy="-1.57 0 -1.57"/>
+      <parent link="world_camera_1"/>
+      <child link="world_camera_link_optical_1"/>
+    </joint>
+    <joint name="world_camera_optical_joint_2" type="fixed">
+      <!-- these values have to be these values otherwise the gazebo camera image
         won't be aligned properly with the frame it is supposedly originating from -->
-     <origin xyz="0 0 0" rpy="-1.57 0 -1.57"/>
-     <parent link="world_camera_2"/>
-     <child link="world_camera_link_optical_2"/>
-   </joint>
-   <joint name="world_camera_optical_joint_3" type="fixed">
-     <!-- these values have to be these values otherwise the gazebo camera image
+      <origin xyz="0 0 0" rpy="-1.57 0 -1.57"/>
+      <parent link="world_camera_2"/>
+      <child link="world_camera_link_optical_2"/>
+    </joint>
+    <joint name="world_camera_optical_joint_3" type="fixed">
+      <!-- these values have to be these values otherwise the gazebo camera image
         won't be aligned properly with the frame it is supposedly originating from -->
-     <origin xyz="0 0 0" rpy="-1.57 0 -1.57"/>
-     <parent link="world_camera_3"/>
-     <child link="world_camera_link_optical_3"/>
-   </joint>
-   <!-- end of joint list -->
+      <origin xyz="0 0 0" rpy="-1.57 0 -1.57"/>
+      <parent link="world_camera_3"/>
+      <child link="world_camera_link_optical_3"/>
+    </joint>
+    <!-- end of joint list -->
     <!-- ROS base_link to ABB World Coordinates transform -->
     <link name="base" />
@@ -496,10 +492,10 @@
      </actuator>
    </transmission>
-  <!-- end of transmission list -->
-  <!-- Fix robot to Gazebo world -->
-  <link name="world"/>
-  <joint name="world_base_link-fixed" type="fixed">
-    <parent link="world"/>
-    <child link="base_link"/>
-  </joint>
+   <!-- end of transmission list -->
+   <!-- Fix robot to Gazebo world -->
+   <link name="world"/>
+   <joint name="world_base_link-fixed" type="fixed">
+     <parent link="world"/>
+     <child link="base_link"/>
+   </joint>
 </robot>

Commit message: more stable grasping

File: irb6640_description/urdf/irb6640.xacro (robot description, xacro)
@@ -157,11 +157,11 @@
         <origin xyz="0 0 0" rpy="0 0 0"/>
         <geometry>
-          <mesh filename="package://irb6640_gazebo/models/vacuum_gripper.dae" scale="0.8 0.8 0.8"/>
-        </geometry>
-      </collision>
-      <visual name="visual">
-        <origin xyz="0 0 0" rpy="0 0 0"/>
-        <geometry>
-          <mesh filename="package://irb6640_gazebo/models/vacuum_gripper.dae" scale="0.8 0.8 0.8"/>
+          <mesh filename="package://irb6640_gazebo/models/vacuum_gripper.dae" scale="0.9 0.9 0.9"/>
+        </geometry>
+      </collision>
+      <visual name="visual">
+        <origin xyz="0 0 0" rpy="0 0 0"/>
+        <geometry>
+          <mesh filename="package://irb6640_gazebo/models/vacuum_gripper.dae" scale="0.9 0.9 0.9"/>
         </geometry>
       </visual>

Commit message: revise inertial of vacuum gripper

File: irb6640_description/urdf/irb6640.xacro (robot description, xacro)
@@ -167,7 +167,7 @@
       </visual>
       <inertial>
-        <mass value="1"/>
+        <mass value="0.4888"/>
         <origin rpy="0 0 0" xyz="0 0 0"/>
-        <inertia ixx="0.1" ixy="0" ixz="0" iyy="0.1" iyz="0" izz="0.1"/>
+        <inertia ixx="0.005856" ixy="0" ixz="0" iyy="0.031721" iyz="0" izz="0.036406"/>
       </inertial>
     </link>
