Commit message: enable joystick teleoperation

File: irb6640_description/urdf/irb6640.xacro (robot description, xacro)
@@ -500,7 +500,7 @@
    </transmission>
    <!-- end of transmission list -->
-   <!-- Fix robot to Gazebo world -->
+   <!-- dummy link to remove warning -->
    <link name="world"/>
-   <joint name="world_base_link-fixed" type="fixed">
+   <joint name="world-base_link-fixed" type="fixed">
      <parent link="world"/>
      <child link="base_link"/>

Commit message: use stl files for collison instead of dae files

File: irb6640_description/urdf/irb6640.xacro (robot description, xacro)
@@ -157,5 +157,5 @@
         <origin xyz="0 0 0" rpy="0 0 0"/>
         <geometry>
-          <mesh filename="package://irb6640_gazebo/models/vacuum_gripper.dae" scale="0.9 0.9 0.9"/>
+          <mesh filename="package://irb6640_gazebo/models/vacuum_gripper.stl" scale="0.9 0.9 0.9"/>
         </geometry>
       </collision>
@@ -246,5 +246,5 @@
         <origin xyz="0 0 0" rpy="0 0 0"/>
         <geometry>
-          <mesh filename="package://irb6640_gazebo/models/camera.dae" scale="0.5 0.5 0.5"/>
+          <mesh filename="package://irb6640_gazebo/models/camera.stl" scale="0.5 0.5 0.5"/>
         </geometry>
       </collision>
@@ -265,5 +265,5 @@
         <origin xyz="0 0 0" rpy="0 0 0"/>
         <geometry>
-	      <mesh filename="package://irb6640_gazebo/models/camera.dae" scale="0.5 0.5 0.5"/>
+	      <mesh filename="package://irb6640_gazebo/models/camera.stl" scale="0.5 0.5 0.5"/>
         </geometry>
       </collision>
@@ -284,5 +284,5 @@
         <origin xyz="0 0 0" rpy="0 0 0"/>
         <geometry>
-	      <mesh filename="package://irb6640_gazebo/models/camera.dae" scale="0.5 0.5 0.5"/>
+	      <mesh filename="package://irb6640_gazebo/models/camera.stl" scale="0.5 0.5 0.5"/>
         </geometry>
       </collision>
